File: design/design/design.kicad_sch (KiCad schematic)
At the start: 18 parts, among them U1 TL084CN, U2 TL084CN, U3 TL084CN

Commit message: feat: PCB routed
Parts:
- added C1: C, Capacitor_THT:C_Disc_D5.0mm_W2.5mm_P5.00mm, symbol Device:C
- added J1: Impulse, Connector_PinHeader_2.54mm:PinHeader_1x02_P2.54mm_Vertical, symbol PCM_SL_Pin_Headers:PINHD_1x2_Male
- added J2: Voltage, Connector_PinHeader_2.54mm:PinHeader_1x03_P2.54mm_Vertical, symbol PCM_SL_Pin_Headers:PINHD_1x3_Male
- added J3: OUT, Connector_PinHeader_2.54mm:PinHeader_1x02_P2.54mm_Vertical, symbol PCM_SL_Pin_Headers:PINHD_1x2_Male
- added L1: L, Inductor_THT:L_Radial_D7.5mm_P3.50mm_Fastron_07P, symbol Device:L
- added R15, R16, R17: R, Resistor_THT:R_Axial_DIN0207_L6.3mm_D2.5mm_P10.16mm_Horizontal, symbol Device:R
- added RV1: 10k, Potentiometer_THT:Potentiometer_Bourns_3296W_Vertical, symbol Device:R_Potentiometer_Trim
- added RV2, RV3: 50k, Potentiometer_THT:Potentiometer_Bourns_3296W_Vertical, symbol Device:R_Potentiometer_Trim
- added U3: TL084CN, PCM_Package_DIP_AKL:DIP-14_W7.62mm_LongPads, symbol PCM_Amplifier_Operational_AKL:TL084CN
- C2, C3: footprint (none) -> Capacitor_THT:C_Disc_D5.0mm_W2.5mm_P5.00mm
- R1, R10, R11, R12, R13, R14, R2, R3, R4, R5, R6, R7, R8: footprint PCM_Package_DIP_AKL:DIP-14_W7.62mm_LongPads -> Resistor_THT:R_Axial_DIN0207_L6.3mm_D2.5mm_P10.16mm_Horizontal
- renumbered U3 to U2
Connections:
- net GND: now also U2.12 (+), C1.1, J1.2, J2.2, J3.2; no longer U2.10 (+)
- net Plant: now also R2.1, U2.14; no longer U2.8
- net VCC: now also U1.4 (V+), J2.1, U3.4 (V+)
- net VEE: now also U1.11 (V-), J2.3, U3.11 (V-)
- net I1: now reaches C3.1, R11.1, R3.1
- net I1: now also U1.1, R16.1; no longer R4.1, U1.8
- net at R11.2, R12.1: now also U1.2 (-); no longer U1.9 (-)
- net FeedBack: now reaches R12.2
- net FeedBack: now also J3.1, U3.6 (-), U3.7
- net P2: now reaches R1.1, U2.1
- net P2: now also RV1.2; no longer R2.1
- net P1: now reaches R3.2, U2.2 (-)
- net P1: now also R15.1; no longer R2.2
- net at R1.2, R10.2, R6.2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: now also U2.13 (-); no longer U2.9 (-)
- net I2: now reaches C2.1, U2.6 (-)
- net I2: now also RV2.2; no longer R4.2
- net D2: now reaches R8.1, U2.8
- net D2: now also RV3.2; no longer R7.1
- net D1: now reaches R5.2, U2.9 (-)
- net D1: now also R17.1; no longer R7.2
- net at R13.1, R14.1: now also U1.3 (+); no longer U1.10 (+)
- net IN: now reaches R13.2
- net IN: now also J1.1
- new net: R16.2, RV2.1
- new net: R7.1, U3.1, U3.2 (-)
- new net: C1.2, L1.2, U3.3 (+)
- new net: R7.2, U3.5 (+)
- new net: R15.2, RV1.1
- new net: R2.2, R4.1
- new net: R17.2, RV3.1
- new net: L1.1, R4.2
- no-connect marks 0 -> 3
Other:
- moved on the sheet: C2, C3, R1, R10, R11, R12, R13, R14, R3, R5, R6, R8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

Commit message: fix: add cap on pcb and design
Parts:
- added C4: C, Capacitor_THT:C_Disc_D5.0mm_W2.5mm_P5.00mm, symbol Device:C
Connections:
- net GND: now also C4.1
- net at R7.2, U3.5 (+): now also C4.2
Other:
- moved on the sheet: R7
Changed lines of the file:
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@@
 	)
 	(junction
+		(at 256.286 64.008)
+		(diameter 0)
+		(color 0 0 0 0)
+	)
+	(junction
 		(at 122.428 28.194)
 		(diameter 0)
@@
 	(wire
 		(pts
+			(xy 256.286 64.77) (xy 256.286 64.008)
+		)
+		(stroke
+			(width 0)
+			(type default)
+		)
+	)
+	(wire
+		(pts
 			(xy 208.788 66.548) (xy 212.09 66.548)
 		)
@@
 	(wire
 		(pts
+			(xy 256.286 74.93) (xy 256.286 72.39)
+		)
+		(stroke
+			(width 0)
+			(type default)
+		)
+	)
+	(wire
+		(pts
 			(xy 146.558 30.734) (xy 146.558 63.754)
 		)
@@
 	(wire
 		(pts
+			(xy 256.286 64.008) (xy 257.302 64.008)
+		)
+		(stroke
+			(width 0)
+			(type default)
+		)
+	)
+	(wire
+		(pts
 			(xy 70.358 47.244) (xy 70.358 61.214)
 		)
@@
 	(wire
 		(pts
-			(xy 255.778 64.008) (xy 257.302 64.008)
+			(xy 255.016 64.008) (xy 256.286 64.008)
 		)
 		(stroke
@@
 	(wire
 		(pts
-			(xy 242.062 64.008) (xy 248.158 64.008)
+			(xy 242.062 64.008) (xy 247.396 64.008)
 		)
 		(stroke
@@
 	)
 	(symbol
+		(lib_id "Device:C")
+		(at 256.286 68.58 180)
+		(unit 1)
+		(body_style 1)
+		(exclude_from_sim no)
+		(in_bom yes)
+		(on_board yes)
+		(in_pos_files yes)
+		(dnp no)
+		(fields_autoplaced yes)
+		(property "Reference" "C4"
+			(at 259.334 67.3099 0)
+			(show_name no)
+			(do_not_autoplace no)
+			(effects
+				(font
+					(size 1.27 1.27)
+				)
+				(justify right)
+			)
+		)
+		(property "Value" "C"
+			(at 259.334 69.8499 0)
+			(show_name no)
+			(do_not_autoplace no)
+			(effects
+				(font
+					(size 1.27 1.27)
+				)
+				(justify right)
+			)
+		)
+		(property "Footprint" "Capacitor_THT:C_Disc_D5.0mm_W2.5mm_P5.00mm"
+			(at 255.3208 64.77 0)
+			(hide yes)
+			(show_name no)
+			(do_not_autoplace no)
+			(effects
+				(font
+					(size 1.27 1.27)
+				)
+			)
+		)
+		(property "Datasheet" ""
+			(at 256.286 68.58 0)
+			(hide yes)
+			(show_name no)
+			(do_not_autoplace no)
+			(effects
+				(font
+					(size 1.27 1.27)
+				)
+			)
+		)
+		(property "Description" "Unpolarized capacitor"
+			(at 256.286 68.58 0)
+			(hide yes)
+			(show_name no)
+			(do_not_autoplace no)
+			(effects
+				(font
+					(size 1.27 1.27)
+				)
+			)
+		)
+		(pin "2"
+		)
+		(pin "1"
+		)
+		(instances
+			(project "design"
+				(path "/bb8eacac-7b7c-407c-b2e2-d96fde64f67b"
+					(reference "C4")
+					(unit 1)
+				)
+			)
+		)
+	)
+	(symbol
 		(lib_id "power:VCC")
 		(at 110.998 20.574 0)
@@
 	)
 	(symbol
+		(lib_id "power:GND")
+		(at 256.286 74.93 0)
+		(mirror y)
+		(unit 1)
+		(body_style 1)
+		(exclude_from_sim no)
+		(in_bom yes)
+		(on_board yes)
+		(in_pos_files yes)
+		(dnp no)
+		(property "Reference" "#PWR013"
+			(at 256.286 81.28 0)
+			(hide yes)
+			(show_name no)
+			(do_not_autoplace no)
+			(effects
+				(font
+					(size 1.27 1.27)
+				)
+			)
+		)
+		(property "Value" "GND"
+			(at 256.286 80.264 0)
+			(show_name no)
+			(do_not_autoplace no)
+			(effects
+				(font
+					(size 1.27 1.27)
+				)
+			)
+		)
+		(property "Footprint" ""
+			(at 256.286 74.93 0)
+			(hide yes)
+			(show_name no)
+			(do_not_autoplace no)
+			(effects
+				(font
+					(size 1.27 1.27)
+				)
+			)
+		)
+		(property "Datasheet" ""
+			(at 256.286 74.93 0)
+			(hide yes)
+			(show_name no)
+			(do_not_autoplace no)
+			(effects
+				(font
+					(size 1.27 1.27)
+				)
+			)
+		)
+		(property "Description" "Power symbol creates a global label with name \"GND\" , ground"
+			(at 256.286 74.93 0)
+			(hide yes)
+			(show_name no)
+			(do_not_autoplace no)
+			(effects
+				(font
+					(size 1.27 1.27)
+				)
+			)
+		)
+		(pin "1"
+		)
+		(instances
+			(project "design"
+				(path "/bb8eacac-7b7c-407c-b2e2-d96fde64f67b"
+					(reference "#PWR013")
+					(unit 1)
+				)
+			)
+		)
+	)
+	(symbol
 		(lib_id "PCM_SL_Pin_Headers:PINHD_1x2_Male")
 		(at 192.024 118.872 0)
@@
 	(symbol
 		(lib_id "Device:R")
-		(at 251.968 64.008 90)
+		(at 251.206 64.008 90)
 		(unit 1)
 		(body_style 1)
@@
 		(fields_autoplaced yes)
 		(property "Reference" "R7"
-			(at 251.968 57.658 90)
+			(at 251.206 57.658 90)
 			(show_name no)
 			(do_not_autoplace no)
@@
 		)
 		(property "Value" "R"
-			(at 251.968 60.198 90)
+			(at 251.206 60.198 90)
 			(show_name no)
 			(do_not_autoplace no)
@@
 		)
 		(property "Footprint" "Resistor_THT:R_Axial_DIN0207_L6.3mm_D2.5mm_P10.16mm_Horizontal"
-			(at 251.968 65.786 90)
+			(at 251.206 65.786 90)
 			(hide yes)
 			(show_name no)
@@
 		)
 		(property "Datasheet" ""
-			(at 251.968 64.008 0)
+			(at 251.206 64.008 0)
 			(hide yes)
 			(show_name no)
@@
 		)
 		(property "Description" "Resistor"
-			(at 251.968 64.008 0)
+			(at 251.206 64.008 0)
 			(hide yes)
 			(show_name no)
