File: design/design/design.kicad_pcb (KiCad board)
At the start: 2 copper layers, 105.3 x 67.6 mm, 29 parts, among them J1 Impulse, J2 Voltage, J3 OUT, U1 TL084CN, U2 TL084CN, U3 TL084CN

Commit message: feat: PCB rearrange
Parts:
- moved J3 60.7 mm to (112.3, 34.3)
- moved J2 28.0 mm to (47.2, 34.3)
- moved R10 16.7 mm to (85.0, 44.2)
- moved C3 10.5 mm to (70.0, 87.5), turned to 0 degrees
- moved L1 9.28 mm to (89.8, 54.5), turned to 0 degrees
- moved R2 8.74 mm to (85.3, 60.3)
- moved R4 8.74 mm to (89.8, 70.5)
- moved R7 7.74 mm to (98.0, 50.4)
- moved C1 7.66 mm to (102.7, 61.8)
- moved U3 7.56 mm to (107.1, 50.4)
- moved R3 3.03 mm to (53.8, 44.5)
- moved R5 2.80 mm to (75.0, 84.6)
- moved R17 2.80 mm to (69.2, 74.4)
- moved R1 2.42 mm to (69.7, 41.7)
- moved R6 2.42 mm to (69.7, 70.5)
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Routing:
- net /FeedBack: track 164.8 -> 211.2 mm
- net VCC: track 222.9 -> 259.5 mm
- net VEE: track 103.7 -> 123.6 mm
- net GND: track 221.2 -> 208.2 mm
- net /I1: track 123.9 -> 112.1 mm
- net /D2: track 47.9 -> 42.6 mm
- net /P1: track 51.4 -> 55.1 mm
- net Net-(C2-Pad2): track 14.2 -> 11.1 mm
- net Net-(U3A--): track 14.7 -> 11.7 mm
- net Net-(R17-Pad2): track 5.68 -> 8.47 mm
- net /D1: track 22.3 -> 20.2 mm
- net /Plant: track 39.8 -> 41.3 mm
- net Net-(U3A-+): track 16.7 -> 15.2 mm
- net /I2: track 39.7 -> 38.3 mm
- net Net-(L1-Pad1): track 4.51 -> 5.78 mm
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
Commit message: chore: minor fixes
Parts:
- moved R11 1.70 mm to (45.6, 41.6)
- moved R12 1.70 mm to (49.4, 51.8)
Routing:
- net GND: track 208.2 -> 224.5 mm
- net VCC: track 259.5 -> 255.1 mm
- net VEE: track 123.6 -> 127.7 mm
- net /I1: track 112.1 -> 108.8 mm
- net Net-(U1A--): track 9.85 -> 8.15 mm
- net /FeedBack: track 211.2 -> 212.7 mm
- net Net-(U3B-+): track 10.3 -> 9.14 mm
- net Net-(U3A-+): track 15.2 -> 15.9 mm

Commit message: fix: add cap on pcb and design
Parts:
- added C4: C, Capacitor_THT:C_Disc_D5.0mm_W2.5mm_P5.00mm, F.Cu at (102.7, 65.4)
Routing:
- net Net-(U3B-+): track 9.14 -> 14.1 mm
- net GND: track 224.5 -> 228.2 mm
Changed lines of the file:
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@@
 		)
 	)
+	(footprint "Capacitor_THT:C_Disc_D5.0mm_W2.5mm_P5.00mm"
+		(layer "F.Cu")
+		(at 102.68 65.4 180)
+		(descr "C, Disc series, Radial, pin pitch=5.00mm, diameter*width=5*2.5mm^2, Capacitor, http://cdn-reichelt.de/documents/datenblatt/B300/DS_KERKO_TC.pdf")
+		(tags "C Disc series Radial pin pitch 5.00mm diameter 5mm width 2.5mm Capacitor")
+		(property "Reference" "C4"
+			(at 2.5 -2.5 0)
+			(layer "F.SilkS")
+			(effects
+				(font
+					(size 1 1)
+					(thickness 0.15)
+				)
+			)
+		)
+		(property "Value" "C"
+			(at 2.5 2.5 0)
+			(layer "F.Fab")
+			(effects
+				(font
+					(size 1 1)
+					(thickness 0.15)
+				)
+			)
+		)
+		(property "Datasheet" ""
+			(at 0 0 0)
+			(layer "F.Fab")
+			(hide yes)
+			(effects
+				(font
+					(size 1.27 1.27)
+				)
+			)
+		)
+		(property "Description" "Unpolarized capacitor"
+			(at 0 0 0)
+			(layer "F.Fab")
+			(hide yes)
+			(effects
+				(font
+					(size 1.27 1.27)
+				)
+			)
+		)
+		(property "KiLib_Generator" "capacitor/THT/other"
+			(at 0 0 0)
+			(layer "F.SilkS")
+			(hide yes)
+			(effects
+				(font
+					(size 1 1)
+					(thickness 0.15)
+				)
+			)
+		)
+		(property ki_fp_filters "C_*")
+		(sheetname "/")
+		(sheetfile "design.kicad_sch")
+		(units
+			(unit
+				(name "A")
+				(pins "1" "2")
+			)
+		)
+		(attr through_hole)
+		(duplicate_pad_numbers_are_jumpers no)
+		(fp_line
+			(start 5.12 1.37)
+			(end -0.12 1.37)
+			(stroke
+				(width 0.12)
+				(type solid)
+			)
+			(layer "F.SilkS")
+		)
+		(fp_line
+			(start 5.12 1.033)
+			(end 5.12 1.37)
+			(stroke
+				(width 0.12)
+				(type solid)
+			)
+			(layer "F.SilkS")
+		)
+		(fp_line
+			(start 5.12 -1.37)
+			(end 5.12 -1.033)
+			(stroke
+				(width 0.12)
+				(type solid)
+			)
+			(layer "F.SilkS")
+		)
+		(fp_line
+			(start -0.12 1.37)
+			(end -0.12 1.033)
+			(stroke
+				(width 0.12)
+				(type solid)
+			)
+			(layer "F.SilkS")
+		)
+		(fp_line
+			(start -0.12 -1.033)
+			(end -0.12 -1.37)
+			(stroke
+				(width 0.12)
+				(type solid)
+			)
+			(layer "F.SilkS")
+		)
+		(fp_line
+			(start -0.12 -1.37)
+			(end 5.12 -1.37)
+			(stroke
+				(width 0.12)
+				(type solid)
+			)
+			(layer "F.SilkS")
+		)
+		(fp_rect
+			(start -1.05 -1.5)
+			(end 6.05 1.5)
+			(stroke
+				(width 0.05)
+				(type solid)
+			)
+			(fill no)
+			(layer "F.CrtYd")
+		)
+		(fp_rect
+			(start 0 -1.25)
+			(end 5 1.25)
+			(stroke
+				(width 0.1)
+				(type solid)
+			)
+			(fill no)
+			(layer "F.Fab")
+		)
+		(fp_text user "${REFERENCE}"
+			(at 2.5 0 0)
+			(layer "F.Fab")
+			(effects
+				(font
+					(size 1 1)
+					(thickness 0.15)
+				)
+			)
+		)
+		(pad "1" thru_hole circle
+			(at 0 0 180)
+			(size 1.6 1.6)
+			(drill 0.8)
+			(layers "*.Cu" "*.Mask")
+			(remove_unused_layers no)
+			(net "GND")
+			(pintype "passive")
+		)
+		(pad "2" thru_hole circle
+			(at 5 0 180)
+			(size 1.6 1.6)
+			(drill 0.8)
+			(layers "*.Cu" "*.Mask")
+			(remove_unused_layers no)
+			(net "Net-(U3B-+)")
+			(pintype "passive")
+		)
+		(embedded_fonts no)
+		(model "${KICAD10_3DMODEL_DIR}/Capacitor_THT.3dshapes/C_Disc_D5.0mm_W2.5mm_P5.00mm.step"
+			(offset
+				(xyz 0 0 0)
+			)
+			(scale
+				(xyz 1 1 1)
+			)
+			(rotate
+				(xyz 0 0 0)
+			)
+		)
+	)
 	(footprint "Resistor_THT:R_Axial_DIN0207_L6.3mm_D2.5mm_P10.16mm_Horizontal"
 		(layer "F.Cu")
@@
 	)
 	(segment
+		(start 102.6661 65.3861)
+		(end 102.68 65.4)
+		(width 0.4)
+		(layer "B.Cu")
+		(net "GND")
+	)
+	(segment
 		(start 115.951472 67.63)
 		(end 111.82 67.63)
@@
 	)
 	(segment
+		(start 102.6661 61.7717)
+		(end 102.6661 65.3861)
+		(width 0.4)
+		(layer "B.Cu")
+		(net "GND")
+	)
+	(segment
 		(start 69.71 59.4)
 		(end 75.7283 59.4)
@@
 	)
 	(segment
+		(start 97.9717 65.1083)
+		(end 97.68 65.4)
+		(width 0.4)
+		(layer "B.Cu")
+		(net "Net-(U3B-+)")
+	)
+	(segment
 		(start 97.9817 60.57)
 		(end 97.9717 60.58)
 		(width 0.4)
 		(layer "B.Cu")
+		(net "Net-(U3B-+)")
+	)
+	(segment
+		(start 97.9717 60.58)
+		(end 97.9717 65.1083)
+		(width 0.4)
+		(layer "B.Cu")

Commit message: chore: minor fixes on traces
Parts:
- moved J2 25.5 mm to (72.7, 34.3)
- moved R2 1.03 mm to (86.3, 60.3)
Routing:
- net VCC: track 255.1 -> 229.9 mm
- net VEE: track 127.7 -> 106.5 mm
- net GND: track 228.2 -> 208.6 mm
- net /FeedBack: track 212.7 -> 217.9 mm
- net Net-(U2D--): track 38.9 -> 41.3 mm
- net /I1: track 108.8 -> 106.7 mm
- net /Plant: track 41.3 -> 43.3 mm
- net /P1: track 55.1 -> 56.4 mm
- net Net-(R2-Pad2): track 4.53 -> 3.50 mm

Commit message: feat: add readme imgs
Other:
- board size 105.3 x 67.6 mm -> 83.6 x 67.6 mm
Changed lines of the file:
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@@
 	(gr_rect
 		(start 36.12 31.76)
-		(end 141.45 99.36)
+		(end 119.75 99.36)
 		(stroke
 			(width 0.05)
@@
 		(polygon
 			(pts
-				(xy 127.79 31.21) (xy 127.79 101.64) (xy 32.75 101.64) (xy 32.75 31.21)
+				(xy 119.75 31.21) (xy 119.75 101.64) (xy 32.75 101.64) (xy 32.75 31.21)
 			)
 		)
